Commit message: Update pmc6r joint moving direction and range

File: pmc6r_support/urdf/pmc6r.urdf.xacro (robot description, xacro)
@@ -111,5 +111,5 @@
         <child link="link_1"/>
         <origin xyz="0.0 0.0 0.423" rpy="0 0 0"/>
-        <axis xyz="0 0 -1"/>
+        <axis xyz="0 0 1"/>
         <limit lower="-2.967" upper="2.967" effort="0" velocity="0.5"/>
     </joint>
@@ -117,7 +117,7 @@
         <parent link="link_1"/>
         <child link="link_2"/>
-        <origin xyz="0.105 0 0" rpy="0 0 0"/>
+        <origin xyz="0.105 0 0" rpy="0 1.5708 0"/>
         <axis xyz="0 -1 0"/>
-        <limit lower="-3.3161" upper="0.7854" effort="0" velocity="0.5"/>
+        <limit lower="-0.7854" upper="3.3161" effort="0" velocity="0.5"/>
     </joint>
     <joint name="joint_3" type="revolute">
@@ -132,5 +132,5 @@
         <child link="link_4"/>
         <origin xyz="0.284 0 0.065" rpy="0 0 0"/>
-        <axis xyz="-1 0 0"/>
+        <axis xyz="1 0 0"/>
         <limit lower="-3.3161" upper="3.3161" effort="0" velocity="0.5"/>
     </joint>
@@ -139,5 +139,5 @@
         <child link="link_5"/>
         <origin xyz="0 0 0" rpy="0 0 0"/>
-        <axis xyz="0 1 0"/>
+        <axis xyz="0 -1 0"/>
         <limit lower="-2.0944" upper="2.0944" effort="0" velocity="0.5"/>
     </joint>

Commit message: Add pmc6r_gazebo package to display mode in Gazebo. Update pmc6r urdf file to work with Gazebo.

File: pmc6r_support/urdf/pmc6r.urdf.xacro (robot description, xacro)
@@ -2,4 +2,25 @@
 <!-- PMC 6-axis Articulated Manipulator -->
 <robot name="pmc6r" xmlns:xacro="http://www.ros.org/wiki/xacro">
+    <!-- Constants for robot dimensions -->
+    <xacro:property name="PI" value="3.1415926535897931"/>
+    <xacro:property name="deg" value="0.017453293"/> <!-- Degrees to Radians -->
+    <!-- assumption value derive from udacity kuka kr210  12:1 -->
+    <xacro:property name="mass0" value="12.5"/> <!-- assumption value for mass -->
+    <xacro:property name="mass1" value="11.5"/> <!-- assumption value for mass -->
+    <xacro:property name="mass2" value="8.0"/> <!-- assumption value for mass -->
+    <xacro:property name="mass3" value="5.9"/> <!-- assumption value for mass -->
+    <xacro:property name="mass4" value="1.5"/> <!-- assumption value for mass -->
+    <xacro:property name="mass5" value="0.6"/> <!-- assumption value for mass -->
+    <xacro:property name="mass6" value="0.04"/> <!-- assumption value for mass -->
+    <!-- Import all Gazebo-customization elements, including Gazebo colors -->
+    <xacro:include filename="$(find pmc6r_support)/urdf/pmc6r.gazebo" />
+    <!-- Add a world link to fix rbot to Gazebo 'base_link' -->
+    <link name="world"/>
+    <joint name="fixed_base_joint" type="fixed">
+        <parent link="world"/>
+        <child link="base_link"/>
+        <origin xyz="0 0 0" rpy="0 0 0"/>
+    </joint>
+    <!-- Start the description of robot -->
     <link name="base_link">
         <visual>
@@ -16,4 +37,12 @@
             </geometry>
         </collision>
+        <inertial>
+            <origin xyz="0 0 0.2" rpy="0 0 0"/>
+            <mass value="${mass0}"/>
+            <inertia
+                ixx="0.6" ixy="0.0" ixz="0.0"
+                iyy="0.7" iyz="0.0"
+                izz="1.0"/>
+        </inertial>
     </link>
     <link name="link_1">
@@ -31,4 +60,12 @@
             </geometry>
         </collision>
+        <inertial>
+            <origin xyz="0.05 0 0.4" rpy="0 0 0"/>
+            <mass value="${mass1}"/>
+            <inertia
+                ixx="0.3" ixy="0.0" ixz="0.0"
+                iyy="0.5" iyz="0.0"
+                izz="0.5"/>
+        </inertial>
     </link>
     <link name="link_2">
@@ -46,4 +83,12 @@
             </geometry>
         </collision>
+        <inertial>
+            <origin xyz="0 0 0.14" rpy="0 0 0"/>
+            <mass value="${mass2}"/>
+            <inertia
+                ixx="0.4" ixy="0.0" ixz="0.0"
+                iyy="0.4" iyz="0.0"
+                izz="0.1"/>
+        </inertial>
     </link>
     <link name="link_3">
@@ -61,4 +106,12 @@
             </geometry>
         </collision>
+        <inertial>
+            <origin xyz="0.07 0 0.03" rpy="0 0 0"/>
+            <mass value="${mass3}"/>
+            <inertia
+                ixx="0.1" ixy="0.0" ixz="0.0"
+                iyy="0.1" iyz="0.0"
+                izz="1.0"/>
+        </inertial>
     </link>
     <link name="link_4">
@@ -76,4 +129,12 @@
             </geometry>
         </collision>
+        <inertial>
+            <origin xyz="0.14 0 0.03" rpy="0 0 0"/>
+            <mass value="${mass4}"/>
+            <inertia
+                ixx="0.0018" ixy="0.0" ixz="0.0"
+                iyy="0.0055" iyz="0.0"
+                izz="0.0064"/>
+        </inertial>
     </link>
     <link name="link_5">
@@ -91,4 +152,12 @@
             </geometry>
         </collision>
+        <inertial>
+            <origin xyz="0 0 0" rpy="0 0 0"/>
+            <mass value="${mass4}"/>
+            <inertia
+                ixx="0.0004" ixy="0.0" ixz="0.0"
+                iyy="0.00068" iyz="0.0"
+                izz="0.00068"/>
+        </inertial>
     </link>
     <link name="link_6">
@@ -106,4 +175,12 @@
             </geometry>
         </collision>
+        <inertial>
+            <origin xyz="0 0 0" rpy="0 0 0"/>
+            <mass value="${mass4}"/>
+            <inertia
+                ixx="0.00004" ixy="0.0" ixz="0.0"
+                iyy="0.00003" iyz="0.0"
+                izz="0.00003"/>
+        </inertial>
     </link>
     <joint name="joint_1" type="revolute">
@@ -113,4 +190,5 @@
         <axis xyz="0 0 1"/>
         <limit lower="-2.967" upper="2.967" effort="0" velocity="0.5"/>
+        <dynamics damping="0.7"/>
     </joint>
     <joint name="joint_2" type="revolute">
@@ -120,4 +198,5 @@
         <axis xyz="0 -1 0"/>
         <limit lower="-0.7854" upper="3.3161" effort="0" velocity="0.5"/>
+        <dynamics damping="0.7"/>
     </joint>
     <joint name="joint_3" type="revolute">
@@ -127,4 +206,5 @@
         <axis xyz="0 -1 0"/>
         <limit lower="-2.0769" upper="2.9496" effort="0" velocity="0.5"/>
+        <dynamics damping="0.7"/>
     </joint>
     <joint name="joint_4" type="revolute">
@@ -134,4 +214,5 @@
         <axis xyz="1 0 0"/>
         <limit lower="-3.3161" upper="3.3161" effort="0" velocity="0.5"/>
+        <dynamics damping="0.7"/>
     </joint>
     <joint name="joint_5" type="revolute">
@@ -141,4 +222,5 @@
         <axis xyz="0 -1 0"/>
         <limit lower="-2.0944" upper="2.0944" effort="0" velocity="0.5"/>
+        <dynamics damping="0.7"/>
     </joint>
     <joint name="joint_6" type="revolute">
@@ -148,4 +230,66 @@
         <axis xyz="1 0 0"/>
         <limit lower="-6.1086" upper="6.1086" effort="0" velocity="0.5"/>
-    </joint>
+        <dynamics damping="0.7"/>
+    </joint>
+    <!--  TODO: Update real gear ratio -->
+    <transmission name="tran1">
+        <type>transmission_interface/SimpleTransmission</type>
+        <joint name="joint_1">
+            <hardwareInterface>PositionJointInterface</hardwareInterface>
+        </joint>
+        <actuator name="motor_1">
+            <hardwareInterface>PositionJointInterface</hardwareInterface>
+            <mechanicalReduction>1</mechanicalReduction>
+        </actuator>
+    </transmission>
+    <transmission name="tran2">
+        <type>transmission_interface/SimpleTransmission</type>
+        <joint name="joint_2">
+            <hardwareInterface>PositionJointInterface</hardwareInterface>
+        </joint>
+        <actuator name="motor_2">
+            <hardwareInterface>PositionJointInterface</hardwareInterface>
+            <mechanicalReduction>1</mechanicalReduction>
+        </actuator>
+    </transmission>
+    <transmission name="tran3">
+        <type>transmission_interface/SimpleTransmission</type>
+        <joint name="joint_3">
+            <hardwareInterface>PositionJointInterface</hardwareInterface>
+        </joint>
+        <actuator name="motor_3">
+            <hardwareInterface>PositionJointInterface</hardwareInterface>
+            <mechanicalReduction>1</mechanicalReduction>
+        </actuator>
+    </transmission>
+    <transmission name="tran4">
+        <type>transmission_interface/SimpleTransmission</type>
+        <joint name="joint_4">
+            <hardwareInterface>PositionJointInterface</hardwareInterface>
+        </joint>
+        <actuator name="motor_4">
+            <hardwareInterface>PositionJointInterface</hardwareInterface>
+            <mechanicalReduction>1</mechanicalReduction>
+        </actuator>
+    </transmission>
+    <transmission name="tran5">
+        <type>transmission_interface/SimpleTransmission</type>
+        <joint name="joint_5">
+            <hardwareInterface>PositionJointInterface</hardwareInterface>
+        </joint>
+        <actuator name="motor_5">
+            <hardwareInterface>PositionJointInterface</hardwareInterface>
+            <mechanicalReduction>1</mechanicalReduction>
+        </actuator>
+    </transmission>
+    <transmission name="tran6">
+        <type>transmission_interface/SimpleTransmission</type>
+        <joint name="joint_6">
+            <hardwareInterface>PositionJointInterface</hardwareInterface>
+        </joint>
+        <actuator name="motor_6">
+            <hardwareInterface>PositionJointInterface</hardwareInterface>
+            <mechanicalReduction>1</mechanicalReduction>
+        </actuator>
+    </transmission>
 </robot>
